Commit message: 更新urdf模型

File: src/nav2_sample/urdf/wc_property.xacro (robot description, xacro)
@@ -3,20 +3,19 @@
   <!-- ****************** ROBOT CONSTANTS *******************************  -->
   <!-- Define the size of the robot's main chassis in meters -->
-  <xacro:property name="base_width" value="0.6" />
-  <xacro:property name="base_length" value="1.18" />
+  <xacro:property name="base_width" value="0.435" />
+  <xacro:property name="base_length" value="1.2" />
   <xacro:property name="base_height" value="0.65" />
   <!-- Define the shape of the robot's two back wheels in meters -->
   <xacro:property name="wheel_radius" value="0.27" />
-  <xacro:property name="wheel_width" value="0.05" />
-  <xacro:property name="front_wheel_radius" value="0.12" />
-  <!-- x-axis points forward, y-axis points to left, z-axis points upwards -->
-  <!-- Define the gap between the wheel and chassis along y-axis in meters -->
-  <xacro:property name="wheel_ygap" value="${wheel_width/2}" />
-  <!-- Position the wheels along the z-axis -->
-  <xacro:property name="wheel_zoff" value="0.2" />
-  <!-- Position the wheels along the x-axis -->
-  <xacro:property name="wheel_xoff" value="0.221" />
-  <!-- Position the caster wheel along the x-axis -->
-  <xacro:property name="caster_xoff" value="-0.40" />
+  <xacro:property name="wheel_width" value="0.08" />
+  <xacro:property name="wheel_ygap" value="${wheel_width/2+0.01}" />
+  <xacro:property name="wheel_zoff" value="0.225" />
+  <xacro:property name="wheel_xoff" value="0.325" />
+  <xacro:property name="front_wheel_radius" value="0.17" />
+  <xacro:property name="s_wheel_radius" value="0.19" />
+  <xacro:property name="s_wheel_width" value="0.08" />
+  <xacro:property name="s_wheel_ygap" value="${-0.002}" />
+  <xacro:property name="s_wheel_zoff" value="${big_wheel_radius+wheel_zoff - s_wheel_radius/2}" />
+  <xacro:property name="s_wheel_xoff" value="${wheel_xoff-0.5}" />
   <!-- Define intertial property macros  -->
   <xacro:macro name="box_inertia" params="m w h d">
@@ -48,17 +47,22 @@
     </material>
   </xacro:macro>
+  <xacro:property name="big_wheel_scale" value="${wheel_radius/0.275}" />
+  <xacro:property name="big_wheel_radius" value="${wheel_radius * big_wheel_scale}" />
+  <xacro:property name="s_wheel_scale" value="${front_wheel_radius/0.1905}" />
+  <xacro:property name="s_wheel_radius" value="${front_wheel_radius * s_wheel_scale}" />
   <!-- <geometry name="wheel_stl">
     <mesh filename="package://nav2_sample/meshes/wheel.STL" scale="${27/29} ${27/29} ${27/29}"/>
   </geometry> -->
   <!-- *********************** DRIVE WHEELS ******************************  -->
-  <xacro:macro name="wheel" params="prefix x_reflect y_reflect wheel_radius wheel_width wheel_xoff wheel_zoff">
+  <xacro:macro name="wheel" params="prefix x_reflect y_reflect">
     <link name="${prefix}_link">
+      <xacro:property name="wheel_scale" value="${wheel_radius/0.275}" />
       <visual>
-        <!-- <origin xyz="${wheel_radius} ${wheel_radius/0.29 * -0.05} ${-wheel_radius}" rpy="0 0 0" /> -->
-        <origin xyz="${y_reflect * wheel_radius} ${ y_reflect * wheel_radius/0.29 * - 0.05} ${-wheel_radius}" rpy="0 0 ${y_reflect * pi/2}" />
-        <geometry>
-          <mesh filename="package://nav2_sample/meshes/wheel.STL" scale="${wheel_radius/0.29} ${wheel_radius/0.29} ${wheel_radius/0.29}"/>
-        </geometry>
-        <material name="light_black" />
+          <origin xyz="0 0 0" rpy="0 0 ${y_reflect * pi/2}" />
+          <geometry>
+            <mesh filename="package://nav2_sample/meshes/wheel2.STL"
+              scale="${wheel_scale} ${wheel_scale} ${wheel_scale}" />
+          </geometry>
+          <material name="light_black" />
       </visual>
       <collision>
@@ -70,11 +74,35 @@
       <xacro:cylinder_inertia m="110.5" r="${wheel_radius}" h="${wheel_width}" />
     </link>
-    <!-- Connect the wheels to the base_link at the appropriate location, and
-       define a continuous joint to allow the wheels to freely rotate about
-       an axis -->
     <joint name="${prefix}_joint" type="revolute">
       <parent link="base_link" />
       <child link="${prefix}_link" />
       <origin xyz="${x_reflect*wheel_xoff} ${y_reflect*(base_width/2+wheel_ygap)} ${-wheel_zoff}"
+        rpy="0 0 0" />
+      <limit upper="3.1415" lower="-3.1415" effort="30" velocity="5.0" />
+      <axis xyz="0 1 0" />
+    </joint>
+  </xacro:macro>
+  <xacro:macro name="samll_wheel" params="prefix x_reflect y_reflect">
+    <link name="${prefix}_link">
+      <visual name="small_wheel">
+        <origin xyz="0 0 0" rpy="0 0 ${y_reflect * pi/2}" />
+        <geometry>
+          <mesh filename="package://nav2_sample/meshes/small_wheel.STL"
+            scale="${s_wheel_scale} ${s_wheel_scale} ${s_wheel_scale}" />
+        </geometry>
+        <material name="light_black" />
+      </visual>
+      <collision>
+        <origin xyz="0 0 0" rpy="${pi/2} 0 0" />
+        <geometry>
+          <cylinder radius="${s_wheel_radius}" length="${s_wheel_width}" />
+        </geometry>
+      </collision>
+      <xacro:cylinder_inertia m="110.5" r="${s_wheel_radius}" h="${s_wheel_width}" />
+    </link>
+    <joint name="${prefix}_joint" type="revolute">
+      <parent link="base_link" />
+      <child link="${prefix}_link" />
+      <origin xyz="${x_reflect*s_wheel_xoff} ${y_reflect*(base_width/2+s_wheel_ygap)} ${-s_wheel_zoff}"
         rpy="0 0 0" />
       <limit upper="3.1415" lower="-3.1415" effort="30" velocity="5.0" />

File: src/nav2_sample/urdf/wheelchair_base.urdf (robot description, URDF)
Before this commit: robot wheelchair_base, 4 links, 3 joints
Links:
- link base_link: geometry collision box size=${base_length} ${base_width} ${base_height}; visual mesh filename=package://nav2_sample/meshes/robot_base.STL scale=1.0 1.0 1.0
Joints:
- joint base_joint: origin xyz=0 0 ${(wheel_radius+wheel_zoff)} rpy=0 0 0 -> xyz=0 0 ${(big_wheel_radius+wheel_zoff)} rpy=0 0 0
- joint imu_joint: origin xyz=0 0 0.30 -> xyz=0 0 0.01; parent base_link -> laser_link
- joint laser_joint: origin xyz=0.0 0.2 0.1 -> xyz=0.0 0.25 0.1
