Commit message: 更新轮椅模型

File: src/nav2_sample/urdf/wheelchair_base.urdf (robot description, URDF)
Before this commit: robot turtlebot3_waffle, 8 links, 7 joints
Links:
- removed link left_small_wheel_link
- removed link left_wheel_link
- removed link right_small_wheel_link
- removed link right_wheel_link
- link base_link: geometry collision box size=${base_length} ${base_width} ${base_height}; visual box size=${base_length} ${base_width} ${base_height}
Joints:
- removed joint left_small_wheel_joint
- removed joint left_wheel_joint
- removed joint right_small_wheel_joint
- removed joint right_wheel_joint
- joint base_joint: origin xyz=0 0 0.54 rpy=0 0 0 -> xyz=0 0 ${(wheel_radius+wheel_zoff)} rpy=0 0 0

Commit message: 初步模拟成功

File: src/nav2_sample/urdf/wheelchair_base.urdf (robot description, URDF)
Before this commit: robot wheelchair_base, 4 links, 3 joints
Links:
- link base_link: geometry collision box size=${base_length} ${base_width} 0.3; visual mesh filename=package://nav2_sample/meshes/robot_base.STL scale=1.0 1.0 1.0
Joints:
- joint base_joint: origin xyz=0 0 ${(big_wheel_radius+wheel_zoff)} rpy=0 0 0 -> xyz=0 0 ${(wheel_radius+wheel_zoff)} rpy=0 0 0
- joint laser_joint: origin xyz=0.0 0.25 0.1 -> xyz=0.0 0.25 0.25

Commit message: 新加入一只小兔

File: src/nav2_sample/urdf/wheelchair_base.urdf (robot description, URDF)
Before this commit: robot wheelchair_base, 4 links, 3 joints
Links:
- added link rabbit_link; visual mesh filename=package://nav2_sample/meshes/rabbit.STL scale=${rabbit_scale} ${rabbit_scale*1.2} ${rabbit_scale}
Joints:
- added joint base_rabbit_joint: type fixed, parent base_link, child rabbit_link, origin xyz=-0.2 0 -0.08
